File: f22-rc-airplane/assets/transmitter/tx-schematic/tx-schematic.kicad_pcb (KiCad board)
At the start: 2 copper layers, 12 parts

Commit message: :memo: more notes
Parts:
- moved NRF24 75.6 mm to (182.3, 76.5)
- moved C4 65.5 mm to (188.0, 139.7), turned to 180 degrees
- moved C2 53.9 mm to (174.6, 74.3), turned to -90 degrees
- moved R3 51.4 mm to (121.9, 132.1)
- moved R4 51.4 mm to (121.9, 116.8)
- moved C3 46.7 mm to (96.6, 139.7), turned to 180 degrees
- moved R1 23.0 mm to (127.0, 121.9), turned to -90 degrees
- moved R2 23.0 mm to (127.0, 106.7), turned to -90 degrees
- moved ESP32 21.0 mm to (139.1, 57.1)
- moved C1 15.9 mm to (119.4, 88.9)
- renumbered C4 to C1, C1 to C2, C2 to C4
Connections:
- MOTOR_JOYSTICK1 pad 1: +3V3 -> GND
- MOTOR_JOYSTICK1 pad 2: GND -> +3V3
- SERVO_JOYSTICK1 pad 1: +3V3 -> GND
- SERVO_JOYSTICK1 pad 2: GND -> +3V3
Routing:
- net GND: track 0.00 -> 71.8 mm
- net Net-(SERVO_JOYSTICK1-VRx): track 0.00 -> 41.4 mm
- net Net-(SERVO_JOYSTICK1-VRy): track 0.00 -> 31.7 mm
- net +3V3: track 0.00 -> 29.5 mm
- net +5V: track 0.00 -> 6.98 mm
- net SERVO_Y_PIN: track 0.00 -> 5.08 mm
- net SERVO_X_PIN : track 0.00 -> 5.08 mm
