File: f22-rc-airplane/assets/transmitter/tx-schematic/tx-schematic.kicad_sch (KiCad schematic)
At the start: 9 parts, among them U1 ESP32-WROOM-32, U2 NRF24L01_Breakout

Commit message: :zap: new F22 TX schematic
Parts:
- removed U1: ESP32-WROOM-32, RF_Module:ESP32-WROOM-32, symbol RF_Module:ESP32-WROOM-32
- removed U3, U4: ~, symbol libs:HW-504
- added C2, C3, C4: 100uF, Capacitor_THT:CP_Radial_D7.5mm_P2.50mm, symbol Device:C_Polarized
- added ESP32: ~, libs:ESP32_30PIN, symbol libs:ESP32_30PIN
- added MOTOR_JOYSTICK1, SERVO_JOYSTICK1: ~, libs:HW-504, symbol libs:HW-504
- C1: footprint (none) -> Capacitor_THT:CP_Radial_D7.5mm_P2.50mm
- R1: renamed from R4; footprint (none) -> Resistor_THT:R_Axial_DIN0207_L6.3mm_D2.5mm_P10.16mm_Horizontal
- R2: renamed from R1; footprint (none) -> Resistor_THT:R_Axial_DIN0207_L6.3mm_D2.5mm_P10.16mm_Horizontal
- R3: footprint (none) -> Resistor_THT:R_Axial_DIN0207_L6.3mm_D2.5mm_P10.16mm_Horizontal
- R4: renamed from R2; footprint (none) -> Resistor_THT:R_Axial_DIN0207_L6.3mm_D2.5mm_P10.16mm_Horizontal
- renumbered U2 to NRF24
Connections:
- net +3V3: now also C2.1, C3.1, ESP32.30 (3V3), MOTOR_JOYSTICK1.1 (GND), SERVO_JOYSTICK1.1 (GND)
- net GND: now also C2.2, C3.2, C4.2, ESP32.14 (GND), ESP32.29 (GND), MOTOR_JOYSTICK1.2 (+5V), SERVO_JOYSTICK1.2 (+5V)
- net NRF24_CE: now also ESP32.25 (RX2)
- net NRF24_CSN: now also ESP32.24 (TX2)
- net NRF24_MISO: now also ESP32.21 (D19)
- net NRF24_MOSI: now also ESP32.16 (D23)
- net NRF24_SCK: now also ESP32.22 (D18)
- net at R1.2: now also SERVO_JOYSTICK1.3 (VRx)
- net at R3.1: now also SERVO_JOYSTICK1.4 (VRy)
- net JOYSTICK_X_PIN  renamed SERVO_X_PIN 
- net JOYSTICK_Y_PIN renamed SERVO_Y_PIN
- net SERVO_Y_PIN: now also ESP32.5 (D35)
- new net +5V: C4.1, ESP32.15 (VIN)
- new net MOTOR_BUTTON_PIN: ESP32.9 (D26), MOTOR_JOYSTICK1.5 (SW)
- new net MOTOR_X_PIN: ESP32.6 (D32)
- new net MOTOR_X_PIN : MOTOR_JOYSTICK1.3 (VRx)
- new net MOTOR_Y_PIN: ESP32.7 (D33), MOTOR_JOYSTICK1.4 (VRy)
- new net SERVO_BUTTON_PIN: ESP32.8 (D25), SERVO_JOYSTICK1.5 (SW)
- new net SERVO_X_PIN: ESP32.4 (D34)
- no-connect marks 29 -> 16
Other:
- moved on the sheet: C1, NRF24, R1, R2, R3, R4

Commit message: :memo: more notes
Parts:
- renumbered C4 to C1, C1 to C2, C2 to C4
Connections:
- net +3V3: now also MOTOR_JOYSTICK1.2 (+5V), SERVO_JOYSTICK1.2 (+5V); no longer MOTOR_JOYSTICK1.1 (GND), SERVO_JOYSTICK1.1 (GND)
- net GND: now also MOTOR_JOYSTICK1.1 (GND), SERVO_JOYSTICK1.1 (GND); no longer MOTOR_JOYSTICK1.2 (+5V), SERVO_JOYSTICK1.2 (+5V)
Other:
- moved on the sheet: C3
